File: Flying_FOCer.kicad_sch (KiCad schematic)
At the start: 54 parts, among them J1 JST-GH, J2 JST-GH, J3 USB_C_Receptacle_USB2.0_16P, J4 Conn_ARM_SWD_TagConnect_TC203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, J5 JST-GH, U1 TCAN3414, U14 TLV70033_SOT353, U15 TLV70033_SOT353, U2 TCAN3414, U3 TPSM5601, U4 STM32G474CEUx, Y1 32MHz

Commit message: Changed Lib link and added BGA part
Parts:
- removed U1, U2: TCAN3414, Package_SO:SOIC-8_3.9x4.9mm_P1.27mm, symbol My Library:TCAN3414
- removed U3: TPSM5601, Package_DFN_QFN:Texas_B3QFN-14-1EP_5x5.5mm_P0.65mm_ThermalVia, symbol My Library:TPSM53603RDA
- added C15, C16, C17, C18, C19, C20, C21, C22, C23, C24, C25, C26, C27, C28, C29, C30, C31, C32, C33, C34: 10µ, Capacitor_SMD:C_1210_3225Metric, symbol Device:C
- added D2: D_Zener, symbol Device:D_Zener
- added J1: Conn_01x06, Connector_JST:JST_GH_SM06B-GHS-TB_1x06-1MP_P1.25mm_Horizontal, symbol Connector_Generic:Conn_01x06
- added R1: R, symbol Device:R
- added RN1, RN2: R_Pack03, symbol Device:R_Pack03
- added U1: TPSM5601, Package_DFN_QFN:Texas_B3QFN-14-1EP_5x5.5mm_P0.65mm_ThermalVia, symbol My_Regulator_Buck_Module:TPSM5601
- added U6: STM32G474PCIx, Package_BGA:ST_UFBGA-121_6x6mm_Layout11x11_P0.5mm, symbol MCU_ST_STM32G4:STM32G474PCIx
- J3: footprint Connector_USB:USB_C_Receptacle_G-Switch_GT-USB-7010ASV -> Connector_USB:USB_C_Receptacle_G-Switch_GT-USB-7051x
- Y1: footprint Crystal:Crystal_SMD_3225-4Pin_3.2x2.5mm -> Crystal:Crystal_SMD_2016-4Pin_2.0x1.6mm
- renumbered C10 to C1, C4 to C10, C6 to C11, C8 to C12, C9 to C13, C12 to C14, C3 to C2, C34 to C3, C5 to C35, C7 to C36, C14 to C37, C15 to C38, C1 to C39, C48 to C4, C2 to C40, C11 to C5, C16 to C6, C17 to C7, C18 to C8, C19 to C9, D2 to D1, D1 to D3, D3 to D4, J5 to J2, J1 to J5, J2 to J6, R33 to R10, R1 to R11, R2 to R12, R15 to R13, R11 to R14, R16 to R15, R17 to R16, R4 to R17, R3 to R18, R6 to R19, R9 to R2, R5 to R20, R12 to R3, R10 to R4, R13 to R5, R14 to R6, R34 to R9, U14 to U2, U15 to U3
Connections:
- net +5V: now also R1.2, U1.7 (VOUT), U1.8 (VOUT)
- net +BATT: now also C15.1, C16.1, C17.1, C18.1, C19.1, C20.1, C21.1, C22.1, C23.1, C24.1, C25.1, C26.1, C27.1, C28.1, C29.1, C30.1, C31.1, C32.1, C33.1, C34.1, D2.1 (K), U1.1 (VIN), U1.14 (VIN)
- net GND: now also C15.2, C16.2, C17.2, C18.2, C19.2, C20.2, C21.2, C22.2, C23.2, C24.2, C25.2, C26.2, C27.2, C28.2, C29.2, C30.2, C31.2, C32.2, C33.2, C34.2, D2.2 (A), J1.6 (Pin_6), U1.10 (AGND), U1.15 (PGND)
- net GPIO: now also RN2.1 (R1.1); no longer J2.3 (Pin_3)
- net SIGNAL: now also RN2.3 (R3.1); no longer J2.1 (Pin_1)
- net TELEM: now also RN2.2 (R2.1); no longer J2.2 (Pin_2)
- net at R2.1, R4.2: now also U1.2 (EN)
- net at C1.2, R3.1, R5.2: now also U1.9 (FB)
- new net: J2.1 (Pin_1), RN2.4 (R3.2)
- new net: J2.2 (Pin_2), RN2.5 (R2.2)
- new net: J2.3 (Pin_3), RN2.6 (R1.2)
- new net: J1.2 (Pin_2), RN1.4 (R3.2)
- new net: J1.3 (Pin_3), RN1.5 (R2.2)
- new net: J1.4 (Pin_4), RN1.6 (R1.2)
- new net: J1.5 (Pin_5), R1.1
- new net: U6.B3 (VSS), U6.B8 (VSS), U6.C10 (VSS), U6.E2 (VSS), U6.J2 (VSS), U6.K10 (VSS), U6.K6 (VSS)
- new net HALL_A: RN1.3 (R3.1)
- new net HALL_B: RN1.2 (R2.1)
- new net HALL_C: RN1.1 (R1.1)
- new net MOT_NTC: J1.1 (Pin_1)
Other:
- note added: "60V clamped diode"
